Commit message: fix: rg2 controller

File: dsr_moveit2/dsr_moveit_config_m0609/config/dsr.ros2_control.xacro (robot description, xacro)
@@ -61,4 +61,5 @@
                 </state_interface>
             </joint>
+            <joint name="rg2_mount" type="fixed"></joint>
             <joint name="rg2_finger_joint1">
                 <command_interface name="position"/>
