Commit message: fix: block err msg via fixed joint

File: dsr_description2/xacro/rg2_macro.xacro (robot description, xacro)
@@ -50,5 +50,5 @@
         <origin xyz="0 0 0" rpy="0 -1.5708 1.5708"/>
     </joint>
-    <joint name="${name}_finger_joint1" type="revolute">
+    <joint name="${name}_finger_joint1" type="fixed">
         <parent link="${name}_hand"/>
         <child link="${name}_leftfinger"/>
@@ -57,5 +57,5 @@
         <limit effort="10.6" lower="0.0" upper="1.18" velocity="1.57"/>
     </joint>
-    <joint name="${name}_finger_joint2" type="revolute">
+    <joint name="${name}_finger_joint2" type="fixed">
         <parent link="${name}_hand"/>
         <child link="${name}_rightfinger"/>
