Commit message: feat: integrate m0609 & RG2 in moveit (except for gripper cotroller)

File: dsr_description2/xacro/m0609.urdf.xacro (robot description, xacro)
@@ -24,4 +24,6 @@
      <xacro:include filename="$(find dsr_description2)/xacro/macro.m0609.blue.xacro" />
   </xacro:if>
+  <!-- RG2 Gripper Macro 포함 -->
+  <xacro:include filename="$(find dsr_description2)/xacro/rg2_macro.xacro"/>
   <xacro:m0609 namespace="$(arg namespace)"/>
   <link name="world" />
@@ -47,3 +49,5 @@
     />
   </xacro:unless>
+  <!-- RG2 그리퍼 매크로 호출 -->
+  <xacro:rg2_gripper parent="link_6" name="rg2"/>
 </robot>

File: dsr_moveit2/dsr_moveit_config_m0609/config/dsr.ros2_control.xacro (robot description, xacro)
@@ -61,4 +61,24 @@
                 </state_interface>
             </joint>
+            <joint name="rg2_finger_joint1">
+                <command_interface name="position"/>
+                <state_interface name="position">
+                    <param name="initial_value">${initial_positions['rg2_finger_joint1']}</param>
+                </state_interface>
+                <command_interface name="velocity"/>
+                <state_interface name="velocity">
+                    <param name="initial_value">0.0</param>
+                </state_interface>
+            </joint>
+            <joint name="rg2_finger_joint2">
+                <command_interface name="position"/>
+                <state_interface name="position">
+                    <param name="initial_value">${initial_positions['rg2_finger_joint2']}</param>
+                </state_interface>
+                <command_interface name="velocity"/>
+                <state_interface name="velocity">
+                    <param name="initial_value">0.0</param>
+                </state_interface>
+            </joint>
         </ros2_control>
     </xacro:macro>

File: dsr_moveit2/dsr_moveit_config_m0609/config/m0609.urdf.xacro (robot description, xacro)
@@ -3,7 +3,9 @@
     <xacro:arg name="initial_positions_file" default="initial_positions.yaml" />
     <!-- Import m0609 urdf file -->
-    <xacro:include filename="$(find dsr_description2)/urdf/m0609.urdf" />
+    <!-- <xacro:include filename="$(find dsr_description2)/urdf/m0609.urdf" /> -->
+    <xacro:include filename="$(find dsr_description2)/xacro/m0609.urdf.xacro" />
     <!-- Import m0609 ros2_control description -->
     <xacro:include filename="dsr.ros2_control.xacro" />
-    <xacro:dsr_moveit_ros2_control name="DSRFakeSystem" initial_positions_file="$(arg initial_positions_file)"/>
+    <!-- <xacro:dsr_moveit_ros2_control name="DSRFakeSystem" initial_positions_file="$(arg initial_positions_file)"/> -->
+    <xacro:dsr_moveit_ros2_control name="m0609" initial_positions_file="$(arg initial_positions_file)"/>
 </robot>

Commit message: feat: integrate rg2 controller action node in m0609 moveit

File: dsr_description2/xacro/m0609.urdf.xacro (robot description, xacro)
@@ -24,6 +24,4 @@
      <xacro:include filename="$(find dsr_description2)/xacro/macro.m0609.blue.xacro" />
   </xacro:if>
-  <!-- RG2 Gripper Macro 포함 -->
-  <xacro:include filename="$(find dsr_description2)/xacro/rg2_macro.xacro"/>
   <xacro:m0609 namespace="$(arg namespace)"/>
   <link name="world" />
@@ -49,4 +47,6 @@
     />
   </xacro:unless>
+  <!-- RG2 Gripper Macro 포함 -->
+  <xacro:include filename="$(find dsr_description2)/xacro/rg2_macro.xacro"/>
   <!-- RG2 그리퍼 매크로 호출 -->
   <xacro:rg2_gripper parent="link_6" name="rg2"/>

File: dsr_description2/xacro/rg2_macro.xacro (robot description, xacro)
@@ -50,5 +50,5 @@
         <origin xyz="0 0 0" rpy="0 -1.5708 1.5708"/>
     </joint>
-    <joint name="${name}_finger_joint1" type="fixed">
+    <joint name="${name}_finger_joint1" type="revolute">
         <parent link="${name}_hand"/>
         <child link="${name}_leftfinger"/>
@@ -57,5 +57,5 @@
         <limit effort="10.6" lower="0.0" upper="1.18" velocity="1.57"/>
     </joint>
-    <joint name="${name}_finger_joint2" type="fixed">
+    <joint name="${name}_finger_joint2" type="revolute">
         <parent link="${name}_hand"/>
         <child link="${name}_rightfinger"/>

File: dsr_moveit2/dsr_moveit_config_m0609/config/dsr.ros2_control.xacro (robot description, xacro)
@@ -67,5 +67,4 @@
                     <param name="initial_value">${initial_positions['rg2_finger_joint1']}</param>
                 </state_interface>
-                <command_interface name="velocity"/>
                 <state_interface name="velocity">
                     <param name="initial_value">0.0</param>
@@ -77,5 +76,4 @@
                     <param name="initial_value">${initial_positions['rg2_finger_joint2']}</param>
                 </state_interface>
-                <command_interface name="velocity"/>
                 <state_interface name="velocity">
                     <param name="initial_value">0.0</param>
